File: hardware/01_gd32f150/01_gd32f150.kicad_sch (KiCad schematic)
At the start: 4 parts, among them J2 LeftConn, J3 RightConn, J4 Qwiic_RA, U1 GD32F150GxUx

Commit message: feat>update schematic
Parts:
- added J3: BOOT Jumper, symbol Connector_Generic:Conn_01x03
- added R1: 10K, symbol Device:R_Small
- renumbered J2 to J1, J3 to J2, U1 to U2
Connections:
- net +3.3V: now also J3.1 (Pin_1); no longer U2.5 (VDDA)
- net BOOT: now also R1.1
- net GND: now also J3.3 (Pin_3)
- net OSC_IN: now reaches U2.2 (OSC_IN/PF0)
- net OSC_OUT: now reaches U2.3 (OSC_OUT/PF1)
- new net: J3.2 (Pin_2), R1.2
- new net VDDA: U2.5 (VDDA)
Other:
- added sheet MCUPeripherals (mcuperipherals.kicad_sch)
